File: inspireFly-EPS.kicad_pcb (KiCad board)
At the start: 4 copper layers, 88 x 94.5 mm, 80 parts, among them J1 USB4085-GF-A_REVB, J2 Conn_01x02_Pin, Q10 SQJA62EP-T1_GE3, Q3 SQJA62EP-T1_GE3, Q4 SQJA62EP-T1_GE3, Q5 SQJA62EP-T1_GE3, Q6 SQJA62EP-T1_GE3, Q7 SQJA62EP-T1_GE3, Q8 SQJA62EP-T1_GE3, Q9 SQJA62EP-T1_GE3, U1 STM32U575RIT6, U2 BQ25750RRVR, U3 TCAN332DCNR, U5 INA180A3IDBVT, U6 INA180A3IDBVT, U7 INA180A3IDBVT, U8 TPS63070RNMR, U9 TPS63070RNMR

Commit message: Lots of routing
Parts:
- removed C14: 47uF, inspireFly-EPS-footprints:CAP_EEEFN1J470L
- removed C25: 100nF, Capacitor_SMD:C_0402_1005Metric_Pad0.74x0.62mm_HandSolder
- removed U5: INA180A3IDBVT, inspireFly-EPS-footprints:SOT95P280X145-5N
- added C30: 10uF, Capacitor_SMD:C_0805_2012Metric_Pad1.18x1.45mm_HandSolder, F.Cu at (100.5, 48.0)
- added C31: 22uF, Capacitor_SMD:C_0805_2012Metric_Pad1.18x1.45mm_HandSolder, F.Cu at (105.9, 46.9)
- added C32: 220nF, Capacitor_SMD:C_0402_1005Metric_Pad0.74x0.62mm_HandSolder, F.Cu at (97.2, 45.1)
- added C33: 2.2uF, Capacitor_SMD:C_0402_1005Metric_Pad0.74x0.62mm_HandSolder, F.Cu at (101.3, 54.5)
- added C34: 22uF, Capacitor_SMD:C_0805_2012Metric_Pad1.18x1.45mm_HandSolder, F.Cu at (105.9, 40.6)
- added C35: 22uF, Capacitor_SMD:C_0805_2012Metric_Pad1.18x1.45mm_HandSolder, F.Cu at (43.0, 52.6)
- added C36: 22uF, Capacitor_SMD:C_0805_2012Metric_Pad1.18x1.45mm_HandSolder, F.Cu at (43.0, 49.3)
- added C37: 10uF, Capacitor_SMD:C_0805_2012Metric_Pad1.18x1.45mm_HandSolder, F.Cu at (83.0, 46.3)
- added C38: 10uF, Capacitor_SMD:C_0805_2012Metric_Pad1.18x1.45mm_HandSolder, F.Cu at (90.0, 41.6)
- added C40: 22uF, Capacitor_SMD:C_0805_2012Metric_Pad1.18x1.45mm_HandSolder, F.Cu at (109.0, 40.6)
- added C41: 22uF, Capacitor_SMD:C_0805_2012Metric_Pad1.18x1.45mm_HandSolder, F.Cu at (87.1, 31.6)
- added C42: 22uF, Capacitor_SMD:C_0805_2012Metric_Pad1.18x1.45mm_HandSolder, F.Cu at (89.5, 31.6)
- added C43: 22uF, Capacitor_SMD:C_0805_2012Metric_Pad1.18x1.45mm_HandSolder, F.Cu at (91.8, 31.6)
- added C44: 10uF, Capacitor_SMD:C_0805_2012Metric_Pad1.18x1.45mm_HandSolder, F.Cu at (155.7, 48.7)
- added C45: 10uF, Capacitor_SMD:C_0805_2012Metric_Pad1.18x1.45mm_HandSolder, F.Cu at (155.7, 51.2)
- added C46: 100nF, Capacitor_SMD:C_0805_2012Metric_Pad1.18x1.45mm_HandSolder, F.Cu at (151.1, 39.7)
- added C47: 22uF, Capacitor_SMD:C_0805_2012Metric_Pad1.18x1.45mm_HandSolder, F.Cu at (151.1, 42.7)
- added C48: 22uF, Capacitor_SMD:C_0805_2012Metric_Pad1.18x1.45mm_HandSolder, F.Cu at (151.1, 45.7)
- added C49: 22uF, Capacitor_SMD:C_0805_2012Metric_Pad1.18x1.45mm_HandSolder, F.Cu at (151.1, 48.7)
- added C50: 22uF, Capacitor_SMD:C_0805_2012Metric_Pad1.18x1.45mm_HandSolder, F.Cu at (42.9, 55.9)
- added JP1: BAT_ENABLE, Jumper:SolderJumper-2_P1.3mm_Open_RoundedPad1.0x1.5mm, F.Cu at (52.5, 31.3)
- added Q1: SQJ123ELP-T1_GE3, inspireFly-EPS-footprints:TRANS_SQJA62EP-T1_GE3, F.Cu at (44.7, 38.8)
- added R25: 115k, Resistor_SMD:R_0402_1005Metric_Pad0.72x0.64mm_HandSolder, F.Cu at (98.6, 54.5)
- added R26: 180k, Resistor_SMD:R_0402_1005Metric_Pad0.72x0.64mm_HandSolder, F.Cu at (103.9, 52.2)
- added R27: 40k, Resistor_SMD:R_0402_1005Metric_Pad0.72x0.64mm_HandSolder, F.Cu at (103.9, 53.4)
- added R28: 40k, Resistor_SMD:R_0402_1005Metric_Pad0.72x0.64mm_HandSolder, F.Cu at (90.8, 43.2)
- added R29: 210k, Resistor_SMD:R_0402_1005Metric_Pad0.72x0.64mm_HandSolder, F.Cu at (90.8, 44.4)
- added R30: 40k, Resistor_SMD:R_0402_1005Metric_Pad0.72x0.64mm_HandSolder, F.Cu at (159.5, 50.9)
- added R31: 210k, Resistor_SMD:R_0402_1005Metric_Pad0.72x0.64mm_HandSolder, F.Cu at (159.5, 52.9)
- added R32: 200k, Resistor_SMD:R_0402_1005Metric_Pad0.72x0.64mm_HandSolder, F.Cu at (159.5, 54.9)
- added U4: MAX77504AAFC+T, inspireFly-EPS-footprints:21-100406_F122A2F&plus_2_MXM, F.Cu at (100.2, 51.8)
- C39: footprint Capacitor_SMD:C_0805_2012Metric_Pad1.18x1.45mm_HandSolder -> Capacitor_SMD:C_0402_1005Metric_Pad0.74x0.62mm_HandSolder
- R15: value 5m -> 47k; footprint Resistor_SMD:R_1206_3216Metric_Pad1.30x1.75mm_HandSolder -> Resistor_SMD:R_0603_1608Metric_Pad0.98x0.95mm_HandSolder
- moved R15 114.1 mm to (50.6, 34.4), turned to 90 degrees
- moved C27 81.9 mm to (72.0, 91.9), turned to 180 degrees
- moved R16 77.2 mm to (89.2, 37.9), turned to 90 degrees
- moved L3 75.9 mm to (85.4, 39.9)
- moved R22 74.7 mm to (71.4, 90.6)
- moved U8 73.6 mm to (87.1, 45.2), turned to 90 degrees
- moved C39 72.8 mm to (88.2, 48.1)
- moved C24 72.6 mm to (84.7, 30.5)
- moved U6 70.8 mm to (83.4, 34.1)
- moved C26 57.4 mm to (96.7, 86.6)
- moved L2 57.3 mm to (101.8, 43.3)
- moved R17 49.1 mm to (96.7, 83.8)
- moved C17 32.6 mm to (77.4, 51.7), turned to 90 degrees
- moved R11 15.5 mm to (58.2, 81.6)
- moved R10 15.5 mm to (58.2, 79.0)
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Connections:
- C17 pad 1: Net-(Q10-S) -> BAT -
- C17 pad 2: BAT - -> V_PROTECTED
- C29 pad 1: ADC1_IN5 -> ADC1_IN3
- L2 pad 2: Net-(U5-IN+) -> +3.3V
- R15 pad 1: Net-(U5-IN+) -> BAT +
- R15 pad 2: +3.3V -> Net-(JP1-A)
- R24 pad 2: ADC1_IN5 -> ADC1_IN3
- R5 pad 2: BAT + -> Net-(Q1-D)
- R7 pad 2: BAT + -> Net-(Q1-D)
- R8 pad 1: BAT + -> Net-(Q1-D)
- U1 pad 14: ADC1_IN5 -> unconnected-(U1A-PA0-Pad14)
- U9 pad 1: unconnected-(U9-PS/SYNC-Pad1) -> V_PROTECTED
- U9 pad 10: unconnected-(U9-PGND-Pad10) -> BAT -
- U9 pad 11: unconnected-(U9-L1-Pad11) -> Net-(U9-L1)
- U9 pad 12_13: unconnected-(U9-VIN-Pad12_13) -> V_PROTECTED
- U9 pad 14: unconnected-(U9-EN-Pad14) -> SUPER_CAP_CHARGE_ENABLE
- U9 pad 15: unconnected-(U9-VSEL-Pad15) -> BAT -
- U9 pad 3: unconnected-(U9-VAUX-Pad3) -> Net-(U9-VAUX)
- U9 pad 4: unconnected-(U9-GND-Pad4) -> BAT -
- U9 pad 5: unconnected-(U9-FB-Pad5) -> Net-(U9-FB)
- U9 pad 6: unconnected-(U9-FB2-Pad6) -> BAT -
- U9 pad 7_8: unconnected-(U9-VOUT-Pad7_8) -> +9V
- U9 pad 9: unconnected-(U9-L2-Pad9) -> Net-(U9-L2)
Routing:
- net Net-(Q1-D): track 0.00 -> 72.1 mm, vias 0 -> 2
- net +3.3V: track 60.1 -> 100.4 mm, vias 0 -> 6
- net BAT +: track 52.7 -> 19.3 mm, vias 2 -> 0
- net Net-(JP1-A): track 0.00 -> 12.6 mm
- net REGEN: track 20.4 -> 8.26 mm
- net Net-(U6-IN+): track 0.00 -> 10.6 mm
- net USB_CC1: track 84.3 -> 75.0 mm
- net Net-(U4-BST): track 0.00 -> 7.67 mm, vias 0 -> 2
- net Net-(U8-L1): track 0.00 -> 6.04 mm
- net Net-(U8-FB): track 0.00 -> 5.14 mm
- net Net-(U8-L2): track 0.00 -> 4.94 mm
- net ADC1_IN4: track 0.00 -> 4.88 mm
- net BAT -: track 49.2 -> 53.0 mm, vias 13 -> 11
- net Net-(U4-FB): track 0.00 -> 3.20 mm
- net V_PROTECTED: track 49.0 -> 51.0 mm
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- added copper zone on F.Cu, net +3.3V
- added copper zone on In2.Cu, net +3.3V
- added copper zone on F.Cu, net +5V
- added copper zone on In2.Cu, net +5V
- added copper zone on F.Cu, net Net-(Q1-D)
- added copper zone on F.Cu, net Net-(U4-LX)
- added copper zone on F.Cu, net Net-(U6-IN+)

Commit message: Updated STM location
Parts:
- removed C26: 100nF, Capacitor_SMD:C_0402_1005Metric_Pad0.74x0.62mm_HandSolder
- removed R17: 10, Resistor_SMD:R_0603_1608Metric_Pad0.98x0.95mm_HandSolder
- added C14: 100nF, Capacitor_SMD:C_0402_1005Metric_Pad0.74x0.62mm_HandSolder, F.Cu at (51.2, 86.4)
- moved C29 100.8 mm to (51.1, 89.8), turned to 180 degrees
- moved R24 100.0 mm to (45.4, 89.5)
- moved C7 38.0 mm to (51.1, 92.8), turned to 180 degrees
- moved C5 34.8 mm to (57.5, 80.5), turned to 90 degrees
- moved R22 26.0 mm to (45.4, 91.1)
- moved C2 22.8 mm to (63.9, 99.5), turned to -90 degrees
- moved C3 22.8 mm to (58.4, 99.5), turned to -90 degrees
- moved C8 20.9 mm to (51.1, 93.8)
- moved C27 20.9 mm to (51.1, 90.9)
- moved U1 20.5 mm to (61.2, 90.2)
- moved TR1 19.9 mm to (84.9, 96.8), turned to 0 degrees
- moved U3 19.7 mm to (79.6, 98.2)
- moved C9 19.4 mm to (74.9, 98.5)
- moved C1 18.1 mm to (70.1, 84.8)
- moved C4 17.4 mm to (65.0, 99.5), turned to -90 degrees
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Routing:
- net USB_CC2: track 89.6 -> 0.00 mm, vias 1 -> 0
- net USB_D+: track 82.8 -> 0.00 mm, vias 1 -> 0
- net USB_D-: track 82.5 -> 0.00 mm, vias 1 -> 0
- net USB_CC1: track 75.0 -> 0.00 mm, vias 1 -> 0
- net +3.3V: track 100.4 -> 47.5 mm, vias 6 -> 17
- net I2C3-SCL: track 32.4 -> 4.27 mm, vias 2 -> 0
- net I2C3-SDA: track 33.0 -> 6.36 mm
- net ADC1_IN3: track 0.00 -> 10.0 mm, vias 0 -> 2
- net BAT -: track 53.0 -> 45.0 mm, vias 11 -> 7
- net CAN_L: track 0.00 -> 5.46 mm
- net ADC1_IN4: track 4.88 -> 9.66 mm, vias 0 -> 2
- net CAN_H: track 0.00 -> 4.00 mm
- net Net-(U2-FSW_SYNC): track 4.71 -> 3.07 mm
- net Net-(U1B-VCAP): track 4.65 -> 3.04 mm
- net POWER_GOOD: track 7.44 -> 6.28 mm
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
Commit message: Added Dead battery to BQ and other routing changes
Parts:
- removed R10: 5.24k, Resistor_SMD:R_0402_1005Metric_Pad0.72x0.64mm_HandSolder
- removed R11: 30.31k, Resistor_SMD:R_0402_1005Metric_Pad0.72x0.64mm_HandSolder
- added D4: DFLS130L-7, inspireFly-EPS-footprints:DFLS130L7, F.Cu at (78.8, 61.3)
- added D5: DFLS130L-7, inspireFly-EPS-footprints:DFLS130L7, F.Cu at (78.8, 65.2)
- added R33: 10K, Resistor_SMD:R_0402_1005Metric_Pad0.72x0.64mm_HandSolder, F.Cu at (48.5, 67.7)
- added R34: 10K, Resistor_SMD:R_0402_1005Metric_Pad0.72x0.64mm_HandSolder, F.Cu at (48.5, 69.0)
- added TP1: DRV_SUP, TestPoint:TestPoint_Pad_D1.5mm, F.Cu at (84.1, 63.5)
- added TP2: V_PROTECTED, TestPoint:TestPoint_Pad_D1.5mm, F.Cu at (79.1, 41.7)
- added TP3: +5V, TestPoint:TestPoint_Pad_D1.5mm, F.Cu at (95.9, 33.8)
- added TP4: +3V, TestPoint:TestPoint_Pad_D1.5mm, F.Cu at (112.8, 42.8)
- added TP5: V_BAT, TestPoint:TestPoint_Pad_D1.5mm, F.Cu at (42.3, 44.6)
- added TP6: V_COMBINED, TestPoint:TestPoint_Pad_D1.5mm, F.Cu at (79.4, 29.9)
- moved C10 51.3 mm to (49.5, 73.2)
- moved C11 50.4 mm to (49.5, 75.5), turned to 0 degrees
- moved R2 49.5 mm to (49.4, 77.7)
- moved R3 39.7 mm to (49.6, 71.2), turned to 180 degrees
- moved C12 39.4 mm to (53.4, 67.5)
- moved R8 6.69 mm to (71.6, 68.8)
- moved R9 6.69 mm to (71.5, 70.0)
- moved R13 6.67 mm to (71.5, 71.6)
- moved R14 6.67 mm to (71.5, 72.8)
- moved R7 5.78 mm to (72.1, 67.0)
- moved D1 1.85 mm to (69.2, 75.1)
- moved C20 1.19 mm to (71.6, 65.6), turned to 0 degrees
- moved C18 1.16 mm to (71.6, 64.5)
- moved R20 0.67 mm to (65.6, 74.4)
- moved R21 0.67 mm to (65.5, 75.7)
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Connections:
- C22 pad 2: +5V -> Net-(D4-K)
- U2 pad 23: +5V -> Net-(D4-K)
- U2 pad 8: BAT - -> Net-(U2-TS)
Routing:
- net Net-(U6-OUT): track 1.12 -> 89.3 mm, vias 1 -> 4
- net USB_CC1: track 0.00 -> 86.7 mm, vias 0 -> 1
- net USB_CC2: track 0.00 -> 83.5 mm, vias 0 -> 1
- net USB_D+: track 0.00 -> 75.0 mm, vias 0 -> 1
- net USB_D-: track 0.00 -> 74.6 mm, vias 0 -> 1
- net Net-(Q4-D): track 0.00 -> 61.7 mm, vias 0 -> 2
- net Net-(U2-ACP): track 82.4 -> 20.8 mm, vias 2 -> 0
- net Net-(U2-ACN): track 70.0 -> 19.7 mm, vias 2 -> 0
- net REGEN: track 8.26 -> 41.2 mm, vias 2 -> 3
- net Net-(D4-K): track 0.00 -> 27.7 mm
- net CAN_RX: track 0.00 -> 27.6 mm, vias 0 -> 2
- net CAN_TX: track 0.00 -> 26.2 mm
- net I2C3-SDA: track 6.36 -> 26.9 mm, vias 0 -> 2
- net I2C3-SCL: track 4.27 -> 24.7 mm, vias 0 -> 2
- net Net-(U2-TS): track 0.00 -> 20.2 mm, vias 0 -> 2
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Other:
- board text added: "+3.3V"
- board text added: "+5V"
- board text added: "DRV_SUP"
- board text added: "V_BAT"
- board text added: "V_COMBINED"
- board text added: "V_PROTECTED"

Commit message: About ready for proto 1
Parts:
- removed C28: 100nF, Capacitor_SMD:C_0402_1005Metric_Pad0.74x0.62mm_HandSolder
- removed R23: 5m, Resistor_SMD:R_1206_3216Metric_Pad1.30x1.75mm_HandSolder
- removed U7: INA180A3IDBVT, inspireFly-EPS-footprints:SOT95P280X145-5N
- added C25: 100nF, Capacitor_SMD:C_0402_1005Metric_Pad0.74x0.62mm_HandSolder, F.Cu at (47.6, 87.4)
- added C26: 10pF, Capacitor_SMD:C_0402_1005Metric_Pad0.74x0.62mm_HandSolder, F.Cu at (49.8, 82.8)
- added C51: 10pF, Capacitor_SMD:C_0402_1005Metric_Pad0.74x0.62mm_HandSolder, F.Cu at (45.0, 87.3)
- added G***: LOGO, inspireFly-EPS-footprints:inspireFly_Logo_long, F.Cu at (91.7, 115.6)
- added L4: 2.2uH, inspireFly-EPS-footprints:WE-MXGI_4020, F.Cu at (92.0, 61.6)
- added R35: 10K, Resistor_SMD:R_0402_1005Metric_Pad0.72x0.64mm_HandSolder, F.Cu at (50.6, 106.8)
- added R36: 10K, Resistor_SMD:R_0402_1005Metric_Pad0.72x0.64mm_HandSolder, F.Cu at (44.9, 89.0)
- added SW1: SW_Push, inspireFly-EPS-footprints:SW_PTS810_SJM_250_SMTR_LFS, F.Cu at (44.9, 105.7)
- added SW2: SW_Push, inspireFly-EPS-footprints:SW_PTS810_SJM_250_SMTR_LFS, F.Cu at (44.9, 98.3)
- added TP7: +9V, TestPoint:TestPoint_Pad_D1.5mm, F.Cu at (98.3, 62.6)
- added Y1: Crystal_GND2, inspireFly-EPS-footprints:XTAL_TSX-3225_16.0000MF18X-AC0, F.Cu at (45.8, 83.9)
- C46: footprint Capacitor_SMD:C_0805_2012Metric_Pad1.18x1.45mm_HandSolder -> Capacitor_SMD:C_0402_1005Metric_Pad0.74x0.62mm_HandSolder
- moved R30 74.0 mm to (85.6, 53.8), turned to 180 degrees
- moved R32 74.0 mm to (85.5, 57.0)
- moved R31 73.9 mm to (85.6, 55.1)
- moved U9 72.3 mm to (89.5, 56.4), turned to -90 degrees
- moved C45 71.0 mm to (85.1, 59.2), turned to 180 degrees
- moved C47 69.0 mm to (87.6, 69.7), turned to 90 degrees
- moved C48 65.0 mm to (90.6, 69.7), turned to 90 degrees
- moved C46 63.9 mm to (88.7, 53.4), turned to 180 degrees
- moved C49 61.2 mm to (93.6, 69.7), turned to 90 degrees
- moved C44 61.1 mm to (95.1, 56.5)
- moved C10 2.94 mm to (52.1, 71.8)
- moved R2 2.94 mm to (52.0, 76.3)
- moved C11 2.94 mm to (52.1, 74.1)
- moved R3 2.94 mm to (52.2, 69.8)
- moved C12 1.25 mm to (54.6, 67.5)
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Connections:
- BT2 pad 1-: BAT - -> GND
- BT2 pad 2-: BAT - -> GND
- C1 pad 2: BAT - -> GND
- C10 pad 2: BAT - -> GND
- C11 pad 1: BAT - -> GND
- C13 pad 2: BAT - -> GND
- C14 pad 2: BAT - -> GND
- C17 pad 1: BAT - -> V_PROTECTED
- C17 pad 2: V_PROTECTED -> GND
- C18 pad 2: BAT - -> GND
- C19 pad 1: BAT - -> GND
- C2 pad 2: BAT - -> GND
- C22 pad 1: BAT - -> GND
- C23 pad 2: BAT - -> GND
- C24 pad 2: BAT - -> GND
- C27 pad 2: BAT - -> GND
- C29 pad 2: BAT - -> GND
- C3 pad 2: BAT - -> GND
- C30 pad 2: BAT - -> GND
- C31 pad 1: BAT - -> GND
- C33 pad 1: BAT - -> GND
- C34 pad 1: BAT - -> GND
- C35 pad 2: BAT - -> GND
- C36 pad 2: BAT - -> GND
- C37 pad 2: BAT - -> GND
- C38 pad 2: BAT - -> GND
- C39 pad 2: BAT - -> GND
- C4 pad 2: BAT - -> GND
- C40 pad 1: BAT - -> GND
- C41 pad 1: BAT - -> GND
- C42 pad 1: BAT - -> GND
- C43 pad 1: BAT - -> GND
- C44 pad 2: BAT - -> GND
- C45 pad 2: BAT - -> GND
- C46 pad 2: BAT - -> GND
- C47 pad 1: BAT - -> GND
- C48 pad 1: BAT - -> GND
- C49 pad 1: BAT - -> GND
- C5 pad 2: BAT - -> GND
- C50 pad 2: BAT - -> GND
- C6 pad 2: BAT - -> GND
- C7 pad 2: BAT - -> GND
- C8 pad 2: BAT - -> GND
- C9 pad 2: BAT - -> GND
- D1 pad 1: BAT - -> GND
- J1 pad A1: BAT - -> GND
- J1 pad A12: BAT - -> GND
- J1 pad B1: BAT - -> GND
- J1 pad B12: BAT - -> GND
- J1 pad S1: BAT - -> GND
- J1 pad S2: BAT - -> GND
- J1 pad S3: BAT - -> GND
- J1 pad S4: BAT - -> GND
- J2 pad 2: BAT - -> GND
- JP1 pad 2: BAT - -> GND
- Q6 pad 3: BAT - -> GND
- Q8 pad 3: BAT - -> GND
- R12 pad 2: BAT - -> GND
- R13 pad 1: BAT - -> GND
- R14 pad 1: BAT - -> GND
- R25 pad 1: BAT - -> GND
- R27 pad 1: BAT - -> GND
- R28 pad 2: BAT - -> GND
- R30 pad 2: BAT - -> GND
- R34 pad 2: BAT - -> GND
- U1 pad 12: BAT - -> GND
- U1 pad 18: BAT - -> GND
- U1 pad 31: BAT - -> GND
- U1 pad 4: unconnected-(U1A-PC15-OSC32_OUT-Pad4) -> Net-(U1A-PC15-OSC32_OUT)
- U1 pad 47: BAT - -> GND
- U1 pad 5: unconnected-(U1A-PH0-OSC_IN-Pad5) -> PH0-OSC-IN
- U1 pad 60: unconnected-(U1A-PH3-BOOT0-Pad60) -> Net-(U1A-PH3-BOOT0)
- U1 pad 63: BAT - -> GND
- U1 pad 7: unconnected-(U1A-NRST-Pad7) -> Net-(U1A-NRST)
- U2 pad 17: BAT - -> GND
- U2 pad 22: BAT - -> GND
- U2 pad 35: BAT - -> GND
- U2 pad 37: BAT - -> GND
- U2 pad 7: BAT - -> GND
- U3 pad 2: BAT - -> GND
- U4 pad 10: BAT - -> GND
- U4 pad 3: BAT - -> GND
- U4 pad 7: BAT - -> GND
- U6 pad 2: BAT - -> GND
- U8 pad 10: BAT - -> GND
- U8 pad 15: BAT - -> GND
- U8 pad 4: BAT - -> GND
- U8 pad 6: BAT - -> GND
- U9 pad 10: BAT - -> GND
- U9 pad 14: SUPER_CAP_CHARGE_ENABLE -> V_PROTECTED
- U9 pad 15: BAT - -> GND
- U9 pad 4: BAT - -> GND
- U9 pad 6: BAT - -> GND
Routing:
- net GND: track 0.00 -> 51.6 mm, vias 0 -> 9
- net BAT -: track 46.2 -> 0.00 mm, vias 9 -> 0
- net Net-(U1A-PH3-BOOT0): track 0.00 -> 34.6 mm, vias 0 -> 2
- net Net-(C25-Pad2): track 0.00 -> 16.7 mm, vias 0 -> 2
- net PH0-OSC-IN: track 0.00 -> 13.8 mm
- net Net-(U1A-PC15-OSC32_OUT): track 0.00 -> 13.4 mm
- net Net-(U1A-NRST): track 0.00 -> 11.5 mm
- net USB_CC1: track 86.7 -> 78.1 mm
- net Net-(U9-L2): track 0.00 -> 6.80 mm
- net Net-(U9-L1): track 0.00 -> 6.65 mm
- net +3.3V: track 51.4 -> 56.8 mm, vias 18 -> 20
- net Net-(U2-ACN): track 19.7 -> 15.8 mm
- net Net-(U6-OUT): track 89.3 -> 93.1 mm
- net +9V: track 0.00 -> 3.75 mm
- net V_BUS_COMBINED: track 80.5 -> 84.3 mm
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- added copper zone on F.Cu, net +9V
- added copper zone on B.Cu, net GND
- added copper zone on F.Cu, net GND
- added copper zone on In1.Cu, net GND
- removed copper zone on B.Cu, net BAT -
- removed copper zone on F.Cu, net BAT -
- removed copper zone on In1.Cu, net BAT -
Other:
- board text added: "+9V"
- board text added: "BAT+"
- board text added: "BOOT"
- board text added: "Design by inspireFly Avionics Memebers"
- board text added: "GND"
- board text added: "RESET"
- board text added: "inspireFly EPS Main Board Rev A.1 Proto"

Commit message: routing updates
Routing:
- net Net-(U6-OUT): track 93.1 -> 93.7 mm
- net Net-(U2-TS): track 22.4 -> 22.9 mm
Changed lines of the file:
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@@
 	)
 	(via
-		(at 60.68 40.89)
+		(at 60.75 40.16)
 		(size 0.7112)
 		(drill 0.3556)
@@
 	)
 	(segment
-		(start 60.68 40.89)
-		(end 56 40.89)
+		(start 54.72 69.79)
+		(end 55.26 69.79)
 		(width 0.2032)
 		(layer "B.Cu")
@@
 	)
 	(segment
-		(start 55.18 41.71)
-		(end 51.66 41.71)
+		(start 45.45 47.92)
+		(end 45.45 60.52)
 		(width 0.2032)
 		(layer "B.Cu")
@@
 	)
 	(segment
-		(start 45.45 60.52)
-		(end 54.72 69.79)
+		(start 56 40.89)
+		(end 55.18 41.71)
 		(width 0.2032)
 		(layer "B.Cu")
@@
 	)
 	(segment
-		(start 45.45 47.92)
-		(end 45.45 60.52)
+		(start 55.18 41.71)
+		(end 51.66 41.71)
 		(width 0.2032)
 		(layer "B.Cu")
@@
 	)
 	(segment
-		(start 54.72 69.79)
-		(end 55.26 69.79)
+		(start 60.02 40.89)
+		(end 56 40.89)
 		(width 0.2032)
 		(layer "B.Cu")
@@
 	)
 	(segment
-		(start 56 40.89)
-		(end 55.18 41.71)
+		(start 45.45 60.52)
+		(end 54.72 69.79)
+		(width 0.2032)
+		(layer "B.Cu")
+		(net 31)
+	)
+	(segment
+		(start 60.75 40.16)
+		(end 60.02 40.89)
 		(width 0.2032)
 		(layer "B.Cu")
@@
 	)
 	(segment
-		(start 80.58 33.6)
-		(end 81.05 33.13)
+		(start 41.97 89.7125)
+		(end 44.4775 92.22)
 		(width 0.2032)
 		(layer "F.Cu")
@@
 	)
 	(segment
-		(start 41.97 89.7125)
-		(end 44.4775 92.22)
+		(start 80.58 33.6)
+		(end 81.05 33.13)
 		(width 0.2032)
 		(layer "F.Cu")
@@
 	)
 	(segment
-		(start 45.72 77.81)
-		(end 41.97 81.56)
+		(start 48.92 80.27)
+		(end 43.26 80.27)
 		(width 0.2032)
 		(layer "F.Cu")
@@
 	)
 	(segment
-		(start 50.36 77.81)
-		(end 45.72 77.81)
+		(start 41.97 81.56)
+		(end 41.97 89.7125)
 		(width 0.2032)
 		(layer "F.Cu")
@@
 	)
 	(segment
-		(start 74.86 70.69)
-		(end 78.04 70.69)
+		(start 43.26 80.27)
+		(end 41.97 81.56)
 		(width 0.2032)
 		(layer "F.Cu")
@@
 	)
 	(segment
-		(start 81.05 33.13)
-		(end 82.14 33.13)
+		(start 49.93 79.26)
+		(end 48.92 80.27)
 		(width 0.2032)
 		(layer "F.Cu")
@@
 	)
 	(segment
-		(start 41.97 81.56)
-		(end 41.97 89.7125)
+		(start 74.86 70.69)
+		(end 78.04 70.69)
+		(width 0.2032)
+		(layer "F.Cu")
+		(net 104)
+	)
+	(segment
+		(start 81.05 33.13)
+		(end 82.14 33.13)
 		(width 0.2032)
 		(layer "F.Cu")
@@
 	)
 	(via
-		(at 50.36 77.81)
+		(at 49.93 79.26)
 		(size 0.4064)
 		(drill 0.2032)
@@
 	)
 	(segment
-		(start 50.36 76.25)
-		(end 50.36 77.81)
+		(start 49.93 79.26)
+		(end 50.36 78.83)
 		(width 0.2032)
 		(layer "B.Cu")
@@
 	)
 	(segment
-		(start 73.98 71.57)
-		(end 72.69 72.86)
+		(start 72.69 72.86)
+		(end 73.98 71.57)
 		(width 0.2032)
 		(layer "B.Cu")
@@
 	)
 	(segment
-		(start 72.69 72.86)
-		(end 53.75 72.86)
+		(start 53.75 72.86)
+		(end 72.69 72.86)
 		(width 0.2032)
 		(layer "B.Cu")
@@
 	)
 	(segment
-		(start 53.75 72.86)
+		(start 50.36 78.83)
 		(end 50.36 76.25)
 		(width 0.2032)
@@
 	)
 	(segment
+		(start 50.36 76.25)
+		(end 53.75 72.86)
+		(width 0.2032)
+		(layer "B.Cu")
+		(net 104)
+	)
+	(segment
 		(start 88.54 45.9625)
 		(end 89.815 45.9625)
@@
 	)
 	(segment
-		(start 50.59 33.4475)
+		(start 43.46 33.98)
 		(end 50.0575 33.98)
 		(width 0.3048)
@@
 	)
 	(segment
-		(start 50.0575 33.98)
-		(end 44.13 33.98)
+		(start 42.815 34.625)
+		(end 43.46 33.98)
 		(width 0.3048)
 		(layer "F.Cu")
@@
 	)
 	(segment
-		(start 42.815 36.045)
-		(end 42.815 35.295)
+		(start 50.59 33.4475)
+		(end 50.59 32.58)
 		(width 0.3048)
 		(layer "F.Cu")
@@
 	)
 	(segment
-		(start 42.815 35.295)
-		(end 44.13 33.98)
+		(start 50.0575 33.98)
+		(end 50.59 33.4475)
 		(width 0.3048)
 		(layer "F.Cu")
@@
 	)
 	(segment
-		(start 50.59 33.4475)
-		(end 50.59 32.58)
+		(start 50.59 32.58)
+		(end 51.89 31.28)
 		(width 0.3048)
 		(layer "F.Cu")
@@
 	)
 	(segment
-		(start 50.59 32.58)
-		(end 51.89 31.28)
+		(start 42.815 36.045)
+		(end 42.815 34.625)
 		(width 0.3048)
 		(layer "F.Cu")
@@
 	)
 	(segment
-		(start 65.21 72.22)
-		(end 65.27 72.16)
+		(start 65.42 72.36)
+		(end 65.34 72.44)
 		(width 0.127)
 		(layer "B.Cu")
@@
 	)
 	(segment
-		(start 49.75 70.61)
-		(end 51.97 70.61)
+		(start 65.42 72.07)
+		(end 65.42 72.36)
 		(width 0.127)
 		(layer "B.Cu")
@@
 	)
 	(segment
-		(start 51.97 70.61)
+		(start 65.34 72.44)
+		(end 64.06 72.44)
+		(width 0.127)
+		(layer "B.Cu")
+		(net 123)
+	)
+	(segment
+		(start 63.84 72.22)
 		(end 53.58 72.22)
 		(width 0.127)
@@
 	)
 	(segment
-		(start 49.1 69.4)
+		(start 49.75 70.61)
 		(end 49.1 69.96)
 		(width 0.127)
@@
 	)
 	(segment
-		(start 49.1 69.96)
-		(end 49.75 70.61)
+		(start 64.06 72.44)
+		(end 63.84 72.22)
 		(width 0.127)
 		(layer "B.Cu")
@@
 	)
 	(segment
-		(start 65.07 71.72)
-		(end 65.05 71.72)
+		(start 51.97 70.61)
+		(end 49.75 70.61)
 		(width 0.127)
 		(layer "B.Cu")
@@
 	)
 	(segment
-		(start 65.27 71.92)
+		(start 65.05 71.72)
 		(end 65.07 71.72)
 		(width 0.127)
@@
 	)
 	(segment
-		(start 53.58 72.22)
-		(end 65.21 72.22)
+		(start 65.07 71.72)
+		(end 65.42 72.07)
 		(width 0.127)
 		(layer "B.Cu")
@@
 	)
 	(segment
-		(start 65.27 72.16)
-		(end 65.27 71.92)
+		(start 49.1 69.96)
+		(end 49.1 69.4)
+		(width 0.127)
+		(layer "B.Cu")
+		(net 123)
+	)
+	(segment
+		(start 53.58 72.22)
+		(end 51.97 70.61)
 		(width 0.127)
 		(layer "B.Cu")
@@
 	)
 	(segment
+		(start 88.76 55.73518)
+		(end 88.76 55.28)
+		(width 0.2032)
+		(layer "F.Cu")
+		(net 125)
+	)
+	(segment
 		(start 89.51 56.48518)
 		(end 89.22982 56.205)
@@
 		(polygon
 			(pts
-				(xy 53.65 35.88) (xy 53.65 41.41) (xy 61.32 41.41) (xy 61.32 33.59) (xy 60.33 32.6) (xy 58.06 32.6)
+				(xy 53.65 35.88) (xy 53.65 41.03) (xy 61.32 41.03) (xy 61.32 33.59) (xy 60.33 32.6) (xy 58.06 32.6)
 				(xy 57.4 33.26) (xy 57.4 36.05) (xy 53.48 36.05)
 			)
@@
 		(polygon
 			(pts
-				(xy 53.21 41.41) (xy 66.36 41.41) (xy 66.4 41.45) (xy 66.4 44.75) (xy 53.22 44.75) (xy 53.2 44.73)
+				(xy 53.34 41.28) (xy 66.23 41.28) (xy 66.4 41.45) (xy 66.4 44.75) (xy 53.22 44.75) (xy 53.2 44.73)
 				(xy 53.2 41.42)
 			)
