File: inspireFly-EPS.kicad_pcb (KiCad board)
At the start: 4 copper layers, 94 x 87 mm, 133 parts, among them J2 Conn_01x02_Pin, J3 FTSH-107-01-L-DV-K-A, J4 Conn_01x02_Pin, J5 USB4110-GF-A, Q14 SQJA62EP-T1_GE3, Q15 SQJA62EP-T1_GE3, Q16 SQJA62EP-T1_GE3, Q17 SQJA62EP-T1_GE3, SW3 SW_TL1015AF160QG, SW4 SW_TL1015AF160QG, U1 BQ25173DSGR, U10 BQ25756ERRVR, U13 TPS259472ARPWR, U3 TCAN332DCNR, U4 MAX77504AAFC+T, U5 STM32U575CIT6, U6 INA180A3IDBVT, U8 TPS63070RNMR, U9 TPS63070RNMR, Y2 XTAL_ABS07-32.768KHZ-T

Commit message: Added 3D step files
Parts:
- moved U1 2.93 mm to (98.0, 73.0)
Changed lines of the file:
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@@
 	(footprint "inspireFly-EPS-footprints:DSG0008A-IPC_B"
 		(layer "F.Cu")
-		(at 99.003033 75.749998)
+		(at 98 73)
 		(tags "BQ25173DSGR ")
 		(property "Reference" "U1"
@@
 		)
 		(embedded_fonts no)
+		(model "${KIPRJMOD}/3D Files/DSG0008A.stp"
+			(offset
+				(xyz 0 0 0)
+			)
+			(scale
+				(xyz 1 1 1)
+			)
+			(rotate
+				(xyz 0 0 0)
+			)
+		)
 	)
 	(footprint "Package_TO_SOT_SMD:SOT-23-8"
@@
 		)
 		(embedded_fonts no)
-		(model "C:/Users/jackf/Downloads/SuperCapacitor_CType.step"
+		(model "${KIPRJMOD}/3D Files/SuperCapacitor_CType.step"
 			(offset
 				(xyz 0 0 0.5)
@@
 		)
 		(embedded_fonts no)
-		(model "C:/Users/jackf/Downloads/SuperCapacitor_CType.step"
+		(model "${KIPRJMOD}/3D Files/SuperCapacitor_CType.step"
 			(offset
 				(xyz 0 0 0.5)
@@
 	)
 	(segment
+		(start 38.655 65.81)
+		(end 38.375 65.53)
+		(width 0.2032)
+		(layer "F.Cu")
+		(net "BQ2_STAT")
+	)
+	(segment
+		(start 38.655 67.19)
+		(end 38.655 65.81)
+		(width 0.2032)
+		(layer "F.Cu")
+		(net "BQ2_STAT")
+	)
+	(segment
+		(start 37.67 67.19)
+		(end 37.665 67.195)
+		(width 0.2032)
+		(layer "F.Cu")
+		(net "BQ2_STAT")
+	)
+	(segment
+		(start 38.655 67.19)
+		(end 37.67 67.19)
+		(width 0.2032)
+		(layer "F.Cu")
+		(net "BQ2_STAT")
+	)
+	(segment
+		(start 37.7475 78.14)
+		(end 37.7475 76.4375)
+		(width 0.1524)
+		(layer "F.Cu")
+		(net "BQ2_STAT")
+	)
+	(segment
+		(start 44.33 72.58)
+		(end 44.33 74.39)
+		(width 0.1524)
+		(layer "F.Cu")
+		(net "BQ2_STAT")
+	)
+	(segment
+		(start 37.665 67.195)
+		(end 37.66 67.2)
+		(width 0.2032)
+		(layer "F.Cu")
+		(net "BQ2_STAT")
+	)
+	(segment
+		(start 37.7475 76.4375)
+		(end 37.77 76.415)
+		(width 0.1524)
+		(layer "F.Cu")
+		(net "BQ2_STAT")
+	)
+	(via
+		(at 44.85 74.55)
+		(size 0.45)
+		(drill 0.3)
+		(layers "F.Cu" "B.Cu")
+		(free yes)
+		(net "BQ2_STAT")
+	)
+	(via
+		(at 43.1 74.56)
+		(size 0.45)
+		(drill 0.3)
+		(layers "F.Cu" "B.Cu")
+		(free yes)
+		(net "BQ2_STAT")
+	)
+	(via
+		(at 45.57 74.56)
+		(size 0.45)
+		(drill 0.3)
+		(layers "F.Cu" "B.Cu")
+		(free yes)
+		(net "BQ2_STAT")
+	)
+	(via
+		(at 42.21 74.56)
+		(size 0.45)
+		(drill 0.3)
+		(layers "F.Cu" "B.Cu")
+		(free yes)
+		(net "BQ2_STAT")
+	)
+	(via
+		(at 37.665 67.195)
+		(size 0.45)
+		(drill 0.3)
+		(layers "F.Cu" "B.Cu")
+		(net "BQ2_STAT")
+	)
+	(via
+		(at 43.96 74.55)
+		(size 0.45)
+		(drill 0.3)
+		(layers "F.Cu" "B.Cu")
+		(free yes)
+		(net "BQ2_STAT")
+	)
+	(via
+		(at 46.46 74.56)
+		(size 0.45)
+		(drill 0.3)
+		(layers "F.Cu" "B.Cu")
+		(free yes)
+		(net "BQ2_STAT")
+	)
+	(segment
 		(start 84.7075 57.29)
 		(end 84.7075 56.7575)
@@
 		(net "Net-(U9-VAUX)")
 	)
-	(segment
-		(start 38.655 65.81)
-		(end 38.375 65.53)
-		(width 0.2032)
-		(layer "F.Cu")
-		(net "BQ2_STAT")
-	)
-	(segment
-		(start 38.655 67.19)
-		(end 38.655 65.81)
-		(width 0.2032)
-		(layer "F.Cu")
-		(net "BQ2_STAT")
-	)
-	(segment
-		(start 37.67 67.19)
-		(end 37.665 67.195)
-		(width 0.2032)
-		(layer "F.Cu")
-		(net "BQ2_STAT")
-	)
-	(segment
-		(start 38.655 67.19)
-		(end 37.67 67.19)
-		(width 0.2032)
-		(layer "F.Cu")
-		(net "BQ2_STAT")
-	)
-	(segment
-		(start 37.7475 78.14)
-		(end 37.7475 76.4375)
-		(width 0.1524)
-		(layer "F.Cu")
-		(net "BQ2_STAT")
-	)
-	(segment
-		(start 44.33 72.58)
-		(end 44.33 74.39)
-		(width 0.1524)
-		(layer "F.Cu")
-		(net "BQ2_STAT")
-	)
-	(segment
-		(start 37.665 67.195)
-		(end 37.66 67.2)
-		(width 0.2032)
-		(layer "F.Cu")
-		(net "BQ2_STAT")
-	)
-	(segment
-		(start 37.7475 76.4375)
-		(end 37.77 76.415)
-		(width 0.1524)
-		(layer "F.Cu")
-		(net "BQ2_STAT")
-	)
-	(via
-		(at 44.85 74.55)
-		(size 0.45)
-		(drill 0.3)
-		(layers "F.Cu" "B.Cu")
-		(free yes)
-		(net "BQ2_STAT")
-	)
-	(via
-		(at 43.1 74.56)
-		(size 0.45)
-		(drill 0.3)
-		(layers "F.Cu" "B.Cu")
-		(free yes)
-		(net "BQ2_STAT")
-	)
-	(via
-		(at 45.57 74.56)
-		(size 0.45)
-		(drill 0.3)
-		(layers "F.Cu" "B.Cu")
-		(free yes)
-		(net "BQ2_STAT")
-	)
-	(via
-		(at 42.21 74.56)
-		(size 0.45)
-		(drill 0.3)
-		(layers "F.Cu" "B.Cu")
-		(free yes)
-		(net "BQ2_STAT")
-	)
-	(via
-		(at 37.665 67.195)
-		(size 0.45)
-		(drill 0.3)
-		(layers "F.Cu" "B.Cu")
-		(net "BQ2_STAT")
-	)
-	(via
-		(at 43.96 74.55)
-		(size 0.45)
-		(drill 0.3)
-		(layers "F.Cu" "B.Cu")
-		(free yes)
-		(net "BQ2_STAT")
-	)
-	(via
-		(at 46.46 74.56)
-		(size 0.45)
-		(drill 0.3)
-		(layers "F.Cu" "B.Cu")
-		(free yes)
-		(net "BQ2_STAT")
-	)
 	(zone
