File: inspireFly-EPS.kicad_sch (KiCad schematic)
At the start: 128 parts, among them J1 USB4085-GF-A_REVB, J2 Conn_01x02_Pin, J3 FTSH-107-01-L-DV-K-A, Q1 SQJ123ELP-T1_GE3, Q10 SQJA62EP-T1_GE3, Q3 SQJA62EP-T1_GE3, Q4 SQJA62EP-T1_GE3, Q5 SQJA62EP-T1_GE3, Q6 SQJA62EP-T1_GE3, Q7 SQJA62EP-T1_GE3, Q8 SQJA62EP-T1_GE3, Q9 SQJA62EP-T1_GE3, SW1 SW_Push, SW2 SW_Push, SW3 SW_Push, U1 STM32U575RIT6, U2 BQ25750RRVR, U3 TCAN332DCNR, U4 MAX77504AAFC+T, U6 INA180A3IDBVT, U7 INA180A3IDBVT, U8 TPS63070RNMR, U9 TPS63070RNMR, Y1 Crystal_GND2

Commit message: Schematic rework
Parts:
- added C53, C55, C61, C62, C63, C65: 100nF, Capacitor_SMD:C_0402_1005Metric_Pad0.74x0.62mm_HandSolder, symbol Device:C
- added C54, C64: 470nF, Capacitor_SMD:C_0402_1005Metric_Pad0.74x0.62mm_HandSolder, symbol Device:C
- added C57, C58: 4.7uF, Capacitor_SMD:C_0402_1005Metric_Pad0.74x0.62mm_HandSolder, symbol Device:C
- added C59: 1uF, Capacitor_SMD:C_0402_1005Metric_Pad0.74x0.62mm_HandSolder, symbol Device:C
- added C66, C68: 10nF, Capacitor_SMD:C_0402_1005Metric_Pad0.74x0.62mm_HandSolder, symbol Device:C
- added C69, C70, C71, C72, C73, C74, C75, C76, C77, C78, C79: 22uF, Capacitor_SMD:C_0805_2012Metric_Pad1.18x1.45mm_HandSolder, symbol Device:C
- added D3: LTST-S270KRKT, LED_SMD:LED_0603_1608Metric_Pad1.05x0.95mm_HandSolder, symbol Device:LED
- added H1, H2: MountingHole_Pad, MountingHole:MountingHole_2.2mm_M2_Pad_TopBottom, symbol Mechanical:MountingHole_Pad
- added JP2: FTSW EN, inspirefly:SmallJumper, symbol Jumper:Jumper_2_Open
- added L5: 10uH, inspireFly-EPS-footprints:WE-XHMA_1090, symbol Device:L
- added Q14, Q15, Q16, Q17: SQJA62EP-T1_GE3, inspireFly-EPS-footprints:TRANS_SQJA62EP-T1_GE3, symbol Simulation_SPICE:NMOS
- added R10, R53: 390k, Resistor_SMD:R_0402_1005Metric, symbol Device:R_US
- added R11: 110k, Resistor_SMD:R_0402_1005Metric, symbol Device:R_US
- added R17: 47k, Resistor_SMD:R_0402_1005Metric_Pad0.72x0.64mm_HandSolder, symbol Device:R_US
- added R38: 210k, Resistor_SMD:R_0402_1005Metric_Pad0.72x0.64mm_HandSolder, symbol Device:R_US
- added R39, R45, R48, R49, R51: 10, Resistor_SMD:R_0402_1005Metric_Pad0.72x0.64mm_HandSolder, symbol Device:R_US
- added R40: 6.2k, Resistor_SMD:R_0402_1005Metric_Pad0.72x0.64mm_HandSolder, symbol Device:R_US
- added R41: 36k, Resistor_SMD:R_0402_1005Metric_Pad0.72x0.64mm_HandSolder, symbol Device:R_US
- added R42, R50: 5m, Resistor_SMD:R_1206_3216Metric_Pad1.30x1.75mm_HandSolder, symbol Device:R_US
- added R43: 15k, Resistor_SMD:R_0402_1005Metric_Pad0.72x0.64mm_HandSolder, symbol Device:R_US
- added R44: 40k, Resistor_SMD:R_0402_1005Metric_Pad0.72x0.64mm_HandSolder, symbol Device:R_US
- added R46, R47: 10k, Resistor_SMD:R_0402_1005Metric_Pad0.72x0.64mm_HandSolder, symbol Device:R_US
- added R52: 680, Resistor_SMD:R_0402_1005Metric_Pad0.72x0.64mm_HandSolder, symbol Device:R_US
- added U10: BQ25756ERRVR, inspirefly:IC_BQ25756ERRVR, symbol inspirefly:BQ25756ERRVR
- added U13: TPS259472ARPWR, inspirefly:RPW0010A-MFG, symbol inspirefly:TPS259470ARPWR
- C10, C11, C12, C13, C15, C16, C17, C18, C19, C20, C21, C22, C23, C35, C36, C50, D4, D5, JP1, L1, Q1, Q10, Q3, Q4, Q5, Q6, Q7, Q8, Q9, R1, R12, R13, R14, R15, R2, R3, R33, R34, R4, R5, R6, R7, R8, R9, TP1, TP2, TP5, U2: now not fitted
Connections:
- net +3.3V: now also R46.2
- net BAT +: no longer BT1.1+, BT1.2+
- net CAN_RX: no longer J3.14
- net CAN_TX: no longer J3.13
- net GND: now also C53.2, C55.1, C57.2, C58.2, C59.1, C63.2, C65.1, C66.1, C68.1, C69.2, C70.2, C71.2, C72.2, C73.2, C74.2, C75.2, C76.2, C77.2, C78.2, H1.1, H2.1, Q15.3 (S), Q17.3 (S), R11.1, R41.2, R43.2, R44.1, R52.1, R53.2, U10.10 (ILIM_HIZ), U10.17 (PGND), U10.22 (PGND__1), U10.35 (ACOV), U10.37 (PGND__2), U10.7 (~{CE}), U13.8 (GND)
- new net: C75.1, C76.1, Q16.1 (D), R49.2, R50.1
- new net: C57.1, R48.1, U10.23 (DRV_SUP)
- new net: R17.2, R38.1, U10.12 (FB)
- new net: R53.1, U13.2 (OVCSEL)
- new net: JP2.2 (B), R10.1, R11.2, U13.1 (EN_UVLO)
- new net: R17.1, U10.11 (FBG)
- new net: C73.1, C74.1, Q14.1 (D), R42.2, R45.2
- new net: C61.2, U10.26 (BTST1)
- new net: R52.2, U13.9 (ILM)
- new net: R43.1, U10.9 (ICHG)
- new net: C62.2, U10.20 (BTST2)
- new net: R44.2, U10.36 (FSW_SYNC)
- new net: C66.2, U13.10 (ITIMER)
- new net: C68.2, U13.7 (dVdt)
- new net: D3.1 (K), R47.1
- new net: R47.2, U10.6 (~{PG})
- new net ACN: C54.2, C55.2, R45.1, U10.29 (ACN)
- new net ACP: C53.1, C54.1, R39.1, U10.30 (ACP)
- new net BAT+: BT1.1+, BT1.2+, C77.1, C78.1, R10.2, R38.2, R50.2, R51.2, U13.5 (IN)
- new net BATMANG_INT_DIN: R46.1, U10.3 (~{INT})
- new net BAT_HIGH_SIDE_DRIVE: Q16.2 (G), U10.19 (HIDRV2)
- new net BAT_LOW_SIDE_DRIVE: Q17.2 (G), U10.21 (LODRV2)
- new net BAT_SIDE_INDUC: C62.1, L5.2, Q16.3 (S), Q17.1 (D), U10.18 (SW2)
- new net EXTERNAL_HIGH_SIDE_DRIVE: Q14.2 (G), U10.27 (HIDRV1)
- new net EXTERNAL_LOW_SIDE_DRIVE: Q15.2 (G), U10.25 (LODRV1)
- new net EXTERNAL_SIDE_INDUC: C61.1, L5.1, Q14.3 (S), Q15.1 (D), U10.28 (SW1)
- new net EXTERNAL_VOLTAGE: C59.2, C71.1, C72.1, R39.2, R42.1, U10.32 (VAC), U10.33 (VAC__1), U10.34 (ACUV)
- new net FOOTSWITCH: JP2.1 (A)
- new net I2C2_SCL: U10.1 (SCL)
- new net I2C2_SDA: U10.2 (SDA)
- new net PROTECTED_VOLTAGE: C69.1, C70.1, C79.1, U13.6 (OUT)
- new net REGN: C58.1, D3.2 (A), R40.1, R48.2, U10.24 (REGN)
- new net SRN: C64.2, C65.2, R51.1, U10.13 (SRN)
- new net SRP: C63.1, C64.1, R49.1, U10.14 (SRP)
- new net THERMISTOR_FEEDBACK: R40.2, R41.1, U10.8 (TS)
- no-connect marks 15 -> 19
Other:
- note added: "78439369100"
- note added: "Batteries"
- note added: "Battery Managment"
- note added: "Footswitch Logic NO: Floating / NC NC: Ground"
- note added: "Overcurrent 5A as 3334 / 680 = 4.9A"
- note added: "Overvoltage (pin 2) is series to GND with 390K to set at 13.8V"
- note added: "Undervoltage at 5.45V V_UV = (1.2(390k + 110k)) / 110k"
