File: inspireFly-EPS.kicad_sch (KiCad schematic)
At the start: 185 parts, among them J2 Conn_01x02_Pin, J3 FTSH-107-01-L-DV-K-A, J4 Conn_01x02_Pin, J5 USB4110-GF-A, Q1 SQJ123ELP-T1_GE3, Q10 SQJA62EP-T1_GE3, Q14 SQJA62EP-T1_GE3, Q15 SQJA62EP-T1_GE3, Q16 SQJA62EP-T1_GE3, Q17 SQJA62EP-T1_GE3, Q3 SQJA62EP-T1_GE3, Q4 SQJA62EP-T1_GE3, Q5 SQJA62EP-T1_GE3, Q6 SQJA62EP-T1_GE3, Q7 SQJA62EP-T1_GE3, Q8 SQJA62EP-T1_GE3, Q9 SQJA62EP-T1_GE3, SW3 SW_TL1015AF160QG, SW4 SW_TL1015AF160QG, U1 BQ25173DSGR, U10 BQ25756ERRVR, U13 TPS259472ARPWR, U2 BQ25750RRVR, U3 TCAN332DCNR, U4 MAX77504AAFC+T, U5 STM32U575CIT6, U6 INA180A3IDBVT, U7 INA180A3IDBVT, U8 TPS63070RNMR, U9 TPS63070RNMR, Y2 XTAL_ABS07-32.768KHZ-T

Commit message: Finished Linear Charger Schematic
Parts:
- added C51, C52: 1.5F, inspireFly-EPS-footprints:CH3R6155CF-ZJN, symbol Device:C_Polarized
Connections:
- net +3.3V: now also U5.29 (PA8)
- net GND: now also C52.2
- net SUPERCAP_LOAD/SLOWCHARGE: now also C41.1, R55.1, U1.8 (OUT), C51.1
- net BQ2_CE: now reaches U1.3 (CE_N)
- net BQ2_CE: now also U5.15 (PA5)
- new net: C51.2, C52.1
Other:
- moved on the sheet: C34, C41, R35, R36, R55, R56, R57, U1
