File: inspireFly-EPS.kicad_sch (KiCad schematic)
At the start: 187 parts, among them J2 Conn_01x02_Pin, J3 FTSH-107-01-L-DV-K-A, J4 Conn_01x02_Pin, J5 USB4110-GF-A, Q1 SQJ123ELP-T1_GE3, Q10 SQJA62EP-T1_GE3, Q14 SQJA62EP-T1_GE3, Q15 SQJA62EP-T1_GE3, Q16 SQJA62EP-T1_GE3, Q17 SQJA62EP-T1_GE3, Q3 SQJA62EP-T1_GE3, Q4 SQJA62EP-T1_GE3, Q5 SQJA62EP-T1_GE3, Q6 SQJA62EP-T1_GE3, Q7 SQJA62EP-T1_GE3, Q8 SQJA62EP-T1_GE3, Q9 SQJA62EP-T1_GE3, SW3 SW_TL1015AF160QG, SW4 SW_TL1015AF160QG, U1 BQ25173DSGR, U10 BQ25756ERRVR, U13 TPS259472ARPWR, U2 BQ25750RRVR, U3 TCAN332DCNR, U4 MAX77504AAFC+T, U5 STM32U575CIT6, U6 INA180A3IDBVT, U7 INA180A3IDBVT, U8 TPS63070RNMR, U9 TPS63070RNMR, Y2 XTAL_ABS07-32.768KHZ-T

Commit message: Added Supercap charger
Parts:
- removed C34, C41: 1uF, Capacitor_SMD:C_0402_1005Metric_Pad0.74x0.62mm_HandSolder, symbol Device:C
- removed C51, C52: 1.5F, inspireFly-EPS-footprints:CH3R6155CF-ZJN, symbol Device:C_Polarized
- added C1, C34: 1.5F, inspireFly-EPS-footprints:CH3R6155CF-ZJN, symbol Device:C_Polarized
- added C52, C56: 1uF, Capacitor_SMD:C_0402_1005Metric_Pad0.74x0.62mm_HandSolder, symbol Device:C
- added R58: 560k, Resistor_SMD:R_0402_1005Metric_Pad0.72x0.64mm_HandSolder, symbol Device:R_US
- added R59: 100k, Resistor_SMD:R_0402_1005Metric_Pad0.72x0.64mm_HandSolder, symbol Device:R_US
- added R60: 240k, Resistor_SMD:R_0402_1005Metric_Pad0.72x0.64mm_HandSolder, symbol Device:R_US
- R35: value 604 -> 10k
- R36: value 100k -> 10k
- R55: value 806k -> 12k
- R56, R57: value 10k -> 200k
Connections:
- net +3.3V: now also R35.1, R36.1; no longer R56.1, R57.1, U5.29 (PA8)
- net +9V: now also C56.2
- net GND: now also R55.2, R57.2, C34.2, C52.1, C56.1, R59.2; no longer R35.2, R36.2
- net SUPERCAP_LOAD/SLOWCHARGE: now also R56.1, C1.1, C52.2, R60.1; no longer R55.1
- net at U1.2 (ISET): now also R55.1; no longer R35.1
- net SUPERCAP_STAT: now reaches U1.5 (STAT)
- net SUPERCAP_STAT: now also R36.2, U5.16 (PA6); no longer R57.2
- net at R56.2: now also R57.1, C1.2, C34.1; no longer U1.6 (PG_N)
- net SUPERCAP_CE: now reaches U5.14 (PA4)
- net SUPERCAP_CE: now also U1.3 (CE_N)
- net BQ2_CE renamed SUPERCAP_PG
- net SUPERCAP_PG: now also R35.2, U1.6 (PG_N); no longer U1.3 (CE_N)
- new net: R58.1, R59.1, U1.7 (FB)
- new net: R58.2, R60.2

Commit message: Finished Routing
Parts:
- added J6, J7, J8: Conn_01x02_Pin, Connector_PinSocket_2.54mm:PinSocket_1x02_P2.54mm_Vertical, symbol Connector:Conn_01x02_Pin
- C14: now not fitted; now left out of the parts list
- C6: value 1uF -> 10uF; footprint Capacitor_SMD:C_0402_1005Metric_Pad0.74x0.62mm_HandSolder -> Capacitor_SMD:C_0603_1608Metric_Pad1.08x0.95mm_HandSolder
Connections:
- net CAN_RX is gone; now on net CAN_RXD: U3.4 (RXD)
- net CAN_TX is gone; now on net CAN_TXD: U3.1 (TXD)
- net +3.3V: now also J7.1 (Pin_1)
- net +5V: now also J8.1 (Pin_1)
- net GND: now also J6.2 (Pin_2), J7.2 (Pin_2), J8.2 (Pin_2)
- net SUPERCAP_OUT: now also J6.1 (Pin_1)
